Commit message: Update Changes

File: workspace/challenge2_ws/install/localization/share/localization/puzzlebot_jetson_ed_urdf.urdf (robot description, URDF)
Before this commit: robot Puzzlebot Jetson-Lidar Ed., 4 links, 3 joints
Joints:
- joint left_wheel: axis (none) -> 1 1 1; origin xyz=0.0 0.0 0.05 -> xyz=0.05 -0.095 -0.05; type fixed -> continuous
- joint right_wheel: axis (none) -> 1 1 1; origin xyz=0.0 0.0 0.05 -> xyz=0.05 0.095 -0.05; type fixed -> continuous

File: workspace/challenge2_ws/src/localization/urdf/puzzlebot_jetson_ed_urdf.urdf (robot description, URDF)
Before this commit: robot Puzzlebot Jetson-Lidar Ed., 4 links, 3 joints
Joints:
- joint left_wheel: axis (none) -> 0 0 1; origin xyz=0.0 0.0 0.05 -> xyz=0.05 -0.095 -0.05; type fixed -> continuous
- joint right_wheel: axis (none) -> 0 0 1; origin xyz=0.0 0.0 0.05 -> xyz=0.05 0.095 -0.05; type fixed -> continuous
